File: TT.sch (KiCad schematic (older format))
At the start: 174 parts, among them J5 PI_ZERO, P1 CONN_02X05, Q1 Q_NPN_BEC, Q2 Q_NPN_BEC, Q3 Q_NPN_BEC, Q4 Q_NPN_BEC, SW1 SW_PUSH_SMALL_H, SW2 SW_PUSH_SMALL_H, SW3 SW_PUSH_SMALL_H, T1 JACK_QINGPU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

Commit message: .sch cleanup
Other:
- note removed: "changelog:\nMK1: initial - diverses beim display falsch und vergessen.\nMK2: +12V nicht zur drossel geroutet \n Ein GND im JTAG stecker nicht geroutet\n GND plane nicht aktualisiert bevor and factory gesandt. -> reset wird auf gnd gezogen - muss gecuttet werden.. evtl. noch mehr - z.b. vom display oder SDcard\n"
- note removed: "für MK4: boot und res switch added - probleme bei buttoninits machen board unbrauchbar da jtag irgendwie abgeschaltet wird. mit boot0 kann der jtag wieder aktiviert werden.\n-- fertig gezeichnet 26.10.2017\n\nmk4 build: 100k pullup einbauen für EN pin am AP65211 sonst geht der regler kaputt beim einschalten.\n\nmk5: separater linear regualtor für 3V3A \n power out pads für ext brds\n rewiring SDc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"
Changed lines of the file:
@@
 encoding utf-8
 Sheet 1 1
-Title "APU - Audio Processing Unit"
-Date "2017-08-06"
+Title "TT remake"
+Date "2018-08-06"
 Rev "v.1.0"
-Comp "Seismic Industries"
-Comment1 "Cortex M4, with SDcard and 2x2 24bit/96kHz Codec "
+Comp ""
+Comment1 ""
 Comment2 ""
 Comment3 ""
@@
 Text GLabel 5575 12025 2    39   Input ~ 0
 CV2
-Text Notes 14550 4675 0    60   ~ 0
-changelog:\nMK1:	initial - diverses beim display falsch und vergessen.\nMK2: 	+12V nicht zur drossel geroutet \n		 Ein GND im JTAG stecker nicht geroutet\n		 GND plane nicht aktualisiert bevor and factory gesandt. -> reset wird auf gnd gezogen - muss gecuttet werden.. evtl. noch mehr - z.b. vom display oder SDcard\n
-Text Notes 14475 5700 0    60   ~ 0
-für MK4: boot und res switch added - probleme bei buttoninits machen board unbrauchbar da jtag irgendwie abgeschaltet wird. mit boot0 kann der jtag wieder aktiviert werden.\n-- fertig gezeichnet 26.10.2017\n\nmk4 build: 100k pullup einbauen für EN pin am AP65211 sonst geht der regler kaputt beim einschalten.\n\nmk5: 		separater linear regualtor für 3V3A \n					power out pads für ext brds\n					rewiring SDcard für korrekte SPI belegung\nMK5.1:	neuer switcher -> AP65211 ausverkauft -> mp1469\n
 Text GLabel 9325 5050 0    39   Input ~ 0
 BTN1

Commit message: corrected some values and the power inversion of U8
Parts:
- R11, R13, R2, R20, R26, R5: value 200k -> 100k
- R12, R14, R21, R27, R3, R6: value 100k -> 33k
- U5: value (none) -> ~
Connections:
- net +12V: now also U8.4 (V+); no longer U8.11 (V-)
- net -12V: now also U8.11 (V-); no longer U8.4 (V+)
Other:
- note added: "notes - 6.6.2018:\n- changed some resistor values around CV ins -> corrected\n- changed text to right values for DC coupling -> corrected\n- inverted power for U8 - > corrected."
- note added: "omit and bridge the DC decoupling elco's if you want direct coupling. \nmount R35, R36, R49, R51 additionally to compensate/set offsets manually."
- note added: "wPI = 4"
- note added: "wPI = 6"
- note removed: "omit and bridge the DC decoupling elco's if you want direct coupling. \nmount R47-50 additionally to compensate/set offsets manually."
Changed lines of the file:
@@
 P 1725 11125
 F 0 "R2" V 1805 11125 50  0000 C CNN
-F 1 "200k" V 1725 11125 50  0000 C CNN
+F 1 "100k" V 1725 11125 50  0000 C CNN
 F 2 "raffilibkicad:R_0603" V 1655 11125 50  0001 C CNN
 F 3 "" H 1725 11125 50  0001 C CNN
@@
 P 7650 14975
 F 0 "U5" H 7750 14725 50  0000 C CNN
-F 1 "" H 7700 15300 50  0000 C CNN
+F 1 "~" H 7700 15300 50  0000 C CNN
 F 2 "raffilibkicad:SOT-223" H 7650 14975 50  0001 C CNN
 F 3 "0.4" H 7650 14975 50  0001 C CNN
@@
 P 1725 11400
 F 0 "R3" V 1805 11400 50  0000 C CNN
-F 1 "100k" V 1725 11400 50  0000 C CNN
+F 1 "33k" V 1725 11400 50  0000 C CNN
 F 2 "raffilibkicad:R_0603" V 1655 11400 50  0001 C CNN
 F 3 "" H 1725 11400 50  0001 C CNN
@@
 P 4275 11125
 F 0 "R11" V 4355 11125 50  0000 C CNN
-F 1 "200k" V 4275 11125 50  0000 C CNN
+F 1 "100k" V 4275 11125 50  0000 C CNN
 F 2 "raffilibkicad:R_0603" V 4205 11125 50  0001 C CNN
 F 3 "" H 4275 11125 50  0001 C CNN
@@
 P 4275 11400
 F 0 "R12" V 4355 11400 50  0000 C CNN
-F 1 "100k" V 4275 11400 50  0000 C CNN
+F 1 "33k" V 4275 11400 50  0000 C CNN
 F 2 "raffilibkicad:R_0603" V 4205 11400 50  0001 C CNN
 F 3 "" H 4275 11400 50  0001 C CNN
@@
 P 6975 11125
 F 0 "R20" V 7055 11125 50  0000 C CNN
-F 1 "200k" V 6975 11125 50  0000 C CNN
+F 1 "100k" V 6975 11125 50  0000 C CNN
 F 2 "raffilibkicad:R_0603" V 6905 11125 50  0001 C CNN
 F 3 "" H 6975 11125 50  0001 C CNN
@@
 P 6975 11400
 F 0 "R21" V 7055 11400 50  0000 C CNN
-F 1 "100k" V 6975 11400 50  0000 C CNN
+F 1 "33k" V 6975 11400 50  0000 C CNN
 F 2 "raffilibkicad:R_0603" V 6905 11400 50  0001 C CNN
 F 3 "" H 6975 11400 50  0001 C CNN
@@
 P 9525 11125
 F 0 "R26" V 9605 11125 50  0000 C CNN
-F 1 "200k" V 9525 11125 50  0000 C CNN
+F 1 "100k" V 9525 11125 50  0000 C CNN
 F 2 "raffilibkicad:R_0603" V 9455 11125 50  0001 C CNN
 F 3 "" H 9525 11125 50  0001 C CNN
@@
 P 9525 11400
 F 0 "R27" V 9605 11400 50  0000 C CNN
-F 1 "100k" V 9525 11400 50  0000 C CNN
+F 1 "33k" V 9525 11400 50  0000 C CNN
 F 2 "raffilibkicad:R_0603" V 9455 11400 50  0001 C CNN
 F 3 "" H 9525 11400 50  0001 C CNN
@@
 P 1725 12975
 F 0 "R5" V 1805 12975 50  0000 C CNN
-F 1 "200k" V 1725 12975 50  0000 C CNN
+F 1 "100k" V 1725 12975 50  0000 C CNN
 F 2 "raffilibkicad:R_0603" V 1655 12975 50  0001 C CNN
 F 3 "" H 1725 12975 50  0001 C CNN
@@
 P 1725 13250
 F 0 "R6" V 1805 13250 50  0000 C CNN
-F 1 "100k" V 1725 13250 50  0000 C CNN
+F 1 "33k" V 1725 13250 50  0000 C CNN
 F 2 "raffilibkicad:R_0603" V 1655 13250 50  0001 C CNN
 F 3 "" H 1725 13250 50  0001 C CNN
@@
 F 6 "Mouser" H 25  3400 50  0001 C CNN "SPR"
 F 7 "71-RCA0603100KJNEC" H 25  3400 50  0001 C CNN "SPN"
-F 8 "" H 25  3400 50  0001 C CNN "SPURL"
 	1    1725 13250
 	0    1    1    0
@@
 P 4275 12975
 F 0 "R13" V 4355 12975 50  0000 C CNN
-F 1 "200k" V 4275 12975 50  0000 C CNN
+F 1 "100k" V 4275 12975 50  0000 C CNN
 F 2 "raffilibkicad:R_0603" V 4205 12975 50  0001 C CNN
 F 3 "" H 4275 12975 50  0001 C CNN
@@
 P 4275 13250
 F 0 "R14" V 4355 13250 50  0000 C CNN
-F 1 "100k" V 4275 13250 50  0000 C CNN
+F 1 "33k" V 4275 13250 50  0000 C CNN
 F 2 "raffilibkicad:R_0603" V 4205 13250 50  0001 C CNN
 F 3 "" H 4275 13250 50  0001 C CNN
@@
 L TL074 U8
 U 5 1 5AFBA5A0
-P 10650 9675
-F 0 "U8" H 10650 9875 50  0000 L CNN
-F 1 "TL074" H 10650 9475 50  0000 L CNN
-F 2 "raffilibkicad:SOIC-14_N" H 10600 9775 50  0001 C CNN
-F 3 "0.558" H 10700 9875 50  0001 C CNN
-F 4 "Texas Instruments" H 0   0   50  0001 C CNN "MFR"
-F 5 "595-TL074CDR SOIC-14 variant" H 0   0   50  0001 C CNN "MPN"
-F 6 "Mouser" H 0   0   50  0001 C CNN "SPR"
-F 7 "595-TL074CDR" H 0   0   50  0001 C CNN "SPN"
-F 8 "" H 0   0   50  0001 C CNN "SPURL"
-	5    10650 9675
-	1    0    0    -1
+P 10450 9675
+F 0 "U8" H 10450 9875 50  0000 L CNN
+F 1 "TL074" H 10450 9475 50  0000 L CNN
+F 2 "raffilibkicad:SOIC-14_N" H 10400 9775 50  0001 C CNN
+F 3 "0.558" H 10500 9875 50  0001 C CNN
+F 4 "Texas Instruments" H -200 0   50  0001 C CNN "MFR"
+F 5 "595-TL074CDR SOIC-14 variant" H -200 0   50  0001 C CNN "MPN"
+F 6 "Mouser" H -200 0   50  0001 C CNN "SPR"
+F 7 "595-TL074CDR" H -200 0   50  0001 C CNN "SPN"
+F 8 "" H -200 0   50  0001 C CNN "SPURL"
+	5    10450 9675
+	-1   0    0    1
 $EndComp
 $Comp
@@
 BTN2
 Text Notes 14275 9950 0    60   ~ 12
-omit and bridge the DC decoupling elco's if you want direct coupling. \nmount R47-50 additionally to compensate/set offsets manually.
+omit and bridge the DC decoupling elco's if you want direct coupling. \nmount R35, R36, R49, R51 additionally to compensate/set offsets manually.
 Text GLabel 13175 8225 3    39   Input ~ 0
 AREF_-10V
@@
 Connection ~ 9700 5050
 Connection ~ 9700 6575
+Text Notes 7925 4400 0    60   ~ 0
+wPI = 4
+Text Notes 7925 4700 0    60   ~ 0
+wPI = 6
+Text Notes 17625 13050 0    60   ~ 12
+notes - 6.6.2018:\n- changed some resistor values around CV ins -> corrected\n- changed text to right values for DC coupling -> corrected\n- inverted power for U8 - > corrected.
 $EndSCHEMATC

Commit message: CV input stage values tweaked to original
Parts:
- R10, R12, R14, R17, R18, R21, R23, R27, R3, R31, R6, R9: value 33k -> 24k9
Other:
- note added: "notes - 6.6.2018:\n- changed some resistor values around CV ins -> corrected\n- changed text to right values for DC coupling -> corrected\n- inverted power for U8 - > corrected.\n\nnotes - 29.06.18:\n- values around CV in tweaked again, now the same as original -> done"
- note removed: "notes - 6.6.2018:\n- changed some resistor values around CV ins -> corrected\n- changed text to right values for DC coupling -> corrected\n- inverted power for U8 - > corrected."
Changed lines of the file:
@@
 P 2400 11400
 F 0 "R9" V 2480 11400 50  0000 C CNN
-F 1 "33k" V 2400 11400 50  0000 C CNN
+F 1 "24k9" V 2400 11400 50  0000 C CNN
 F 2 "raffilibkicad:R_0603" V 2330 11400 50  0001 C CNN
 F 3 "" H 2400 11400 50  0001 C CNN
@@
 P 4950 11400
 F 0 "R17" V 5030 11400 50  0000 C CNN
-F 1 "33k" V 4950 11400 50  0000 C CNN
+F 1 "24k9" V 4950 11400 50  0000 C CNN
 F 2 "raffilibkicad:R_0603" V 4880 11400 50  0001 C CNN
 F 3 "" H 4950 11400 50  0001 C CNN
@@
 P 7625 11400
 F 0 "R23" V 7705 11400 50  0000 C CNN
-F 1 "33k" V 7625 11400 50  0000 C CNN
+F 1 "24k9" V 7625 11400 50  0000 C CNN
 F 2 "raffilibkicad:R_0603" V 7555 11400 50  0001 C CNN
 F 3 "" H 7625 11400 50  0001 C CNN
@@
 P 10175 11400
 F 0 "R31" V 10255 11400 50  0000 C CNN
-F 1 "33k" V 10175 11400 50  0000 C CNN
+F 1 "24k9" V 10175 11400 50  0000 C CNN
 F 2 "raffilibkicad:R_0603" V 10105 11400 50  0001 C CNN
 F 3 "" H 10175 11400 50  0001 C CNN
@@
 P 1725 11400
 F 0 "R3" V 1805 11400 50  0000 C CNN
-F 1 "33k" V 1725 11400 50  0000 C CNN
+F 1 "24k9" V 1725 11400 50  0000 C CNN
 F 2 "raffilibkicad:R_0603" V 1655 11400 50  0001 C CNN
 F 3 "" H 1725 11400 50  0001 C CNN
@@
 P 4275 11400
 F 0 "R12" V 4355 11400 50  0000 C CNN
-F 1 "33k" V 4275 11400 50  0000 C CNN
+F 1 "24k9" V 4275 11400 50  0000 C CNN
 F 2 "raffilibkicad:R_0603" V 4205 11400 50  0001 C CNN
 F 3 "" H 4275 11400 50  0001 C CNN
@@
 P 6975 11400
 F 0 "R21" V 7055 11400 50  0000 C CNN
-F 1 "33k" V 6975 11400 50  0000 C CNN
+F 1 "24k9" V 6975 11400 50  0000 C CNN
 F 2 "raffilibkicad:R_0603" V 6905 11400 50  0001 C CNN
 F 3 "" H 6975 11400 50  0001 C CNN
@@
 P 9525 11400
 F 0 "R27" V 9605 11400 50  0000 C CNN
-F 1 "33k" V 9525 11400 50  0000 C CNN
+F 1 "24k9" V 9525 11400 50  0000 C CNN
 F 2 "raffilibkicad:R_0603" V 9455 11400 50  0001 C CNN
 F 3 "" H 9525 11400 50  0001 C CNN
@@
 P 2400 13250
 F 0 "R10" V 2480 13250 50  0000 C CNN
-F 1 "33k" V 2400 13250 50  0000 C CNN
+F 1 "24k9" V 2400 13250 50  0000 C CNN
 F 2 "raffilibkicad:R_0603" V 2330 13250 50  0001 C CNN
 F 3 "" H 2400 13250 50  0001 C CNN
@@
 P 4950 13250
 F 0 "R18" V 5030 13250 50  0000 C CNN
-F 1 "33k" V 4950 13250 50  0000 C CNN
+F 1 "24k9" V 4950 13250 50  0000 C CNN
 F 2 "raffilibkicad:R_0603" V 4880 13250 50  0001 C CNN
 F 3 "" H 4950 13250 50  0001 C CNN
@@
 P 1725 13250
 F 0 "R6" V 1805 13250 50  0000 C CNN
-F 1 "33k" V 1725 13250 50  0000 C CNN
+F 1 "24k9" V 1725 13250 50  0000 C CNN
 F 2 "raffilibkicad:R_0603" V 1655 13250 50  0001 C CNN
 F 3 "" H 1725 13250 50  0001 C CNN
@@
 P 4275 13250
 F 0 "R14" V 4355 13250 50  0000 C CNN
-F 1 "33k" V 4275 13250 50  0000 C CNN
+F 1 "24k9" V 4275 13250 50  0000 C CNN
 F 2 "raffilibkicad:R_0603" V 4205 13250 50  0001 C CNN
 F 3 "" H 4275 13250 50  0001 C CNN
@@
 wPI = 6
 Text Notes 17625 13050 0    60   ~ 12
-notes - 6.6.2018:\n- changed some resistor values around CV ins -> corrected\n- changed text to right values for DC coupling -> corrected\n- inverted power for U8 - > corrected.
+notes - 6.6.2018:\n- changed some resistor values around CV ins -> corrected\n- changed text to right values for DC coupling -> corrected\n- inverted power for U8 - > corrected.\n\nnotes - 29.06.18:\n- values around CV in tweaked again, now the same as original -> done
 $EndSCHEMATC
